File: PLACAS/Genus_MainBoard_Lite v.1.0/Genus_MainBoard_Lite-v.1.0.sch (EAGLE design)
At the start: 60 parts, among them U1 FT232RLSSOP, U2 MP2307DN-LF-Z, X1 53398-06, X15 JST-XH-05-PIN-LONG-PAD, X2 JST-XH-08-PIN-ROUND-PAD, X3 USB-SMD-NS, X5 53398-06

Commit message: Add files via upload
Connections:
- new net BOOT: SLOT-1G$1.13, SLOT-2G$1.13
Other:
- note added: "C:/Users/marcu/Desktop/Ensino Superior/Graduação - Eng Elétrica/Zenith/zenith-v2.bmp"
