File: PLACAS/Varella_Feature_Board v.1.0/Varella_Feature_Board v.1.0.brd (EAGLE design)
At the start: 70 x 42.9 mm, 70 parts, among them U1 MAX31856, U3 MAX31856, U4 MAX31856, X1 53261-10, X2 JST-XH-02-PIN-ROUND-PAD, X3 JST-XH-02-PIN-ROUND-PAD, X4 JST-XH-02-PIN-ROUND-PAD, Y2 32768kHz

Commit message: Add files via upload
Connections:
- net 12V(1) renamed 12V_A
- net 12V(2) renamed 12V_B
- removed net N$21: JP1.B43, SJ9.1
- removed net N$22: JP1.B40, SJ10.1
- removed net NSS_BUS: COMM_MICRO1.20, JP1.B15
- removed net SCKL_BUS: COMM_MICRO1.21, JP1.A14
- new net N$1: JP1.A40, JP1.A43, SJ10.1, SJ9.1
- new net SCLK_BUS: COMM_MICRO1.21, JP1.B14
- new net SS_BUS: COMM_MICRO1.20, JP1.A15
- net BOOT: now also JP1.A13; no longer JP1.B13
- net CAN_H: now also JP1.B7; no longer JP1.A7
- net CAN_L: now also JP1.B8; no longer JP1.A8
- net GB1_1: now also SJ3.1; no longer SJ6.2
- net GB1_2: now also SJ6.2; no longer SJ3.1
- net GB1_3: now also SJ4.1; no longer SJ7.2
- net GB1_4: now also SJ5.1; no longer SJ8.2
- net GB1_5: now also SJ7.2; no longer SJ4.1
- net GB1_6: now also SJ8.2; no longer SJ5.1
- net MISO_BUS: now also JP1.B15; no longer JP1.A15
- net MOSI_BUS: now also JP1.A14; no longer JP1.B14
- net NRST: now also JP1.A12; no longer JP1.B12
- net SCL_BUS: now also JP1.B27; no longer JP1.A27
- net SDA_BUS: now also JP1.B26; no longer JP1.A26
- net SWCLK: now also JP1.B11; no longer JP1.A11
- net SWDIO: now also JP1.B12; no longer JP1.A12
- net SWO: now also JP1.B13; no longer JP1.A13
- net UART_RX: now also JP1.A8; no longer JP1.B8
- net UART_TX: now also JP1.A7; no longer JP1.B7
Routing:
- net SS_BUS: track 0.00 -> 26.8 mm, vias 0 -> 1
- net NSS_BUS: track 25.4 -> 0.00 mm
- net SCLK_BUS: track 0.00 -> 16.5 mm, vias 0 -> 2
- net N$1: track 0.00 -> 16.0 mm, vias 0 -> 1
- net SCKL_BUS: track 14.5 -> 0.00 mm, vias 1 -> 0
- net N$21: track 9.57 -> 0.00 mm
- net N$22: track 9.17 -> 0.00 mm
- net SWDIO: track 49.8 -> 53.2 mm, vias 1 -> 2
- net GND: track 46.3 -> 43.6 mm
- net GND(6): track 2.44 -> 0.00 mm
- net !FAULT_1: track 63.7 -> 61.3 mm
- net MISO_BUS: track 15.9 -> 18.3 mm, vias 1 -> 2
- net MOSI_BUS: track 13.2 -> 15.2 mm, vias 2 -> 1
- net N$9: track 9.60 -> 11.6 mm
- net N$20: track 8.01 -> 9.84 mm
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