File: PLACAS/Varella_Feature_Board v.1.0/Varella_Feature_Board v.1.0.sch (EAGLE design)
At the start: 70 parts, among them U1 MAX31856, U3 MAX31856, U4 MAX31856, X1 53261-10, X2 JST-XH-02-PIN-ROUND-PAD, X3 JST-XH-02-PIN-ROUND-PAD, X4 JST-XH-02-PIN-ROUND-PAD, Y2 32768kHz

Commit message: Add files via upload
Connections:
- removed net N$19: JP1.GB1_5, SJ4.2
- removed net N$21: JP1.PWM_2, SJ9.1
- removed net N$22: JP1.PWM_1, SJ10.1
- removed net NSS_BUS: COMM_MICRO1.PA4, JP1.SS_(1)
- removed net SCKL_BUS: COMM_MICRO1.PA5, JP1.SCLK_(1)
- new net N$1: JP1.PWM_1, JP1.PWM_2, SJ10.1, SJ9.1
- new net N$2: JP1.GB1_3, SJ4.2
- new net SCLK_BUS: COMM_MICRO1.PA5, JP1.SCLK_1
- new net SS_BUS: COMM_MICRO1.PA4, JP1.SS_1
- net BOOT: now also JP1.BOOT; no longer JP1.NC_5
- net GB1_1: now also SJ3.1; no longer SJ6.2
- net GB1_2: now also SJ6.2; no longer SJ3.1
- net GB1_3: now also SJ4.1; no longer SJ7.2
- net GB1_4: now also SJ5.1; no longer SJ8.2
- net GB1_5: now also SJ7.2; no longer SJ4.1
- net GB1_6: now also SJ8.2; no longer SJ5.1
- net GND: now also JP1.GND_1, JP1.GND_2, JP1.GND_3; no longer JP1.GND(1), JP1.GND(2), JP1.GND(5)
- net GND(6): now also JP1.GND_4; no longer JP1.GND(6)
- net MISO_BUS: now also JP1.MISO_1; no longer JP1.MISO_(1)
- net MOSI_BUS: now also JP1.MOSI_1; no longer JP1.MOSI_(1)
- net N$15: now also JP1.GB1_5; no longer JP1.GB1_3
- net N$16: now also JP1.GB1_6; no longer JP1.GB1_4
- net N$17: now also JP1.GB1_4; no longer JP1.GB1_6
- net N$20: now also JP1.GB1_1; no longer JP1.GB1_2
- net N$5: now also JP1.5V_A, JP1.5V_B; no longer JP1.5V(1), JP1.5V(2)
- net N$8: now also JP1.3V3_A, JP1.3V3_B; no longer JP1.3V3(1), JP1.3V3(2)
- net N$9: now also JP1.GB1_2; no longer JP1.GB1_1
- net NRST: now also JP1.NRST; no longer JP1.NC_4
- net SCL_BUS: now also JP1.SCL_1; no longer JP1.SCL_(1)
- net SDA_BUS: now also JP1.SDA_1; no longer JP1.SDA_(1)
- net SWCLK: now also JP1.SWCLK; no longer JP1.NC_1
- net SWDIO: now also JP1.SWDIO; no longer JP1.NC_2
- net SWO: now also JP1.SWO; no longer JP1.NC_3
Other:
- moved on the sheet: SJ10, SJ3, SJ4, SJ5, SJ9
