File: Design Blocks/Schematic/FTDI  FT232.sch (EAGLE design)
At the start: 9 parts, among them U1 FT232RLSSOP, X2 USB-SMD-NS

Commit message: dbls
Parts:
- renumbered LED1 to TX, LED2 to RX
Connections:
- net 3.3V renamed +3V3
- net 5V renamed +5V
