File: PLACAS/Sensors_Dev_Breakouts v.1.0 - C/Breakout UVB.sch (EAGLE design)
At the start: 3 parts

Commit message: Add files via upload
Other:
- note added: "1/1"
- note added: "Breakout UVB v.1.0"
- note added: "EESC - USP"
- note added: "Julho de 2020"
- note added: "Júlio Calandrin"
- moved on the sheet: GUVB, JP7, JP8
