File: PLACAS/Sensors_Dev_Breakouts v.1.0 - C/Breakout UVC.brd (EAGLE design)
At the start: 10 x 10 mm, 5 parts

Commit message: Add files via upload
Parts:
- removed JP1, JP2: (no value), pinhead(1x3):1X02
Connections:
- net GND: no longer JP1.1, JP1.2, JP2.1, JP2.2
Routing:
- net GND: track 33.6 -> 8.02 mm
Changed lines of the file:
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@@
 </autorouter>
 <elements>
-<element name="JP1" library="pinhead(1x3)" package="1X02" package3d_urn="urn:adsk.eagle:package:22435/2" value="" x="5" y="0" smashed="yes">
-<attribute name="POPULARITY" value="98" x="21.51" y="-2.54" size="1.778" layer="27" display="off"/>
-<attribute name="VALUE" x="2.46" y="-3.175" size="1.27" layer="27"/>
-</element>
-<element name="JP2" library="pinhead(1x3)" package="1X02" package3d_urn="urn:adsk.eagle:package:22435/2" value="" x="5" y="10" smashed="yes">
-<attribute name="POPULARITY" value="98" x="21.51" y="1.11" size="1.778" layer="27" display="off"/>
-<attribute name="VALUE" x="2.46" y="6.825" size="1.27" layer="27"/>
-</element>
 <element name="U$1" library="GUVX" package="GUV_C" value="GUVC-S10GD" x="2.57" y="3.09" smashed="yes"/>
 <element name="JP5" library="pinhead(1x3)" package="1X02" package3d_urn="urn:adsk.eagle:package:22435/2" value="" x="10" y="5" smashed="yes" rot="R90">
@@
 <signals>
 <signal name="GND">
-<contactref element="JP2" pad="1"/>
-<contactref element="JP2" pad="2"/>
-<contactref element="JP1" pad="1"/>
-<contactref element="JP1" pad="2"/>
 <polygon width="0.1524" layer="1">
 <vertex x="-1.27" y="11.43"/>
@@
 <vertex x="11.43" y="11.43"/>
 </polygon>
-<contactref element="JP5" pad="1"/>
-<contactref element="JP5" pad="2"/>
-<contactref element="U$1" pad="ANODE"/>
-<wire x1="10" y1="6.27" x2="9.652" y2="6.35" width="1.016" layer="1"/>
-<wire x1="10" y1="3.73" x2="9.6504" y2="3.81" width="1.016" layer="1"/>
-<wire x1="6.086375" y1="2.676625" x2="6.223" y2="2.54" width="0.8128" layer="1"/>
-<wire x1="3.73" y1="0" x2="3.81" y2="2.54" width="0.8128" layer="1"/>
-<wire x1="6.35" y1="3.81" x2="6.27" y2="0" width="0.8128" layer="1"/>
-<wire x1="6.27" y1="10" x2="6.3508" y2="10.1592" width="0.8128" layer="1"/>
-<wire x1="6.3508" y1="10.1592" x2="6.3508" y2="6.35" width="0.8128" layer="1"/>
-<wire x1="3.73" y1="10" x2="3.81" y2="7.62" width="0.8128" layer="1"/>
-<wire x1="10" y1="3.73" x2="6.35" y2="3.81" width="0.8128" layer="1"/>
-<wire x1="10" y1="6.27" x2="6.3508" y2="6.35" width="0.8128" layer="1"/>
 <polygon width="0.0762" layer="16">
 <vertex x="-1" y="11"/>
@@
 <vertex x="11" y="11"/>
 </polygon>
-<wire x1="3.73" y1="10" x2="3.73" y2="8.27" width="1.016" layer="16"/>
-<wire x1="3.73" y1="8.27" x2="4" y2="8" width="1.016" layer="16"/>
-<wire x1="6.27" y1="10" x2="6.27" y2="8.27" width="1.016" layer="16"/>
-<wire x1="6.27" y1="8.27" x2="6" y2="8" width="1.016" layer="16"/>
-<wire x1="10" y1="6.27" x2="8.27" y2="6.27" width="1.016" layer="16"/>
-<wire x1="8.27" y1="6.27" x2="8" y2="6" width="1.016" layer="16"/>
-<wire x1="10" y1="3.73" x2="8.27" y2="3.73" width="1.016" layer="16"/>
-<wire x1="8.27" y1="3.73" x2="8" y2="4" width="1.016" layer="16"/>
-<wire x1="6.27" y1="0" x2="6.27" y2="1.73" width="1.016" layer="16"/>
-<wire x1="6.27" y1="1.73" x2="6" y2="2" width="1.016" layer="16"/>
-<wire x1="3.73" y1="0" x2="3.73" y2="1.73" width="1.016" layer="16"/>
-<wire x1="3.73" y1="1.73" x2="4" y2="2" width="1.016" layer="16"/>
+<contactref element="JP5" pad="1"/>
+<contactref element="JP5" pad="2"/>
+<contactref element="U$1" pad="ANODE"/>
+<wire x1="10" y1="6.27" x2="9.652" y2="6.35" width="1.016" layer="1"/>
+<wire x1="10" y1="3.73" x2="9.6504" y2="3.81" width="1.016" layer="1"/>
+<wire x1="10" y1="3.73" x2="6.35" y2="3.81" width="0.8128" layer="1"/>
+<wire x1="10" y1="6.27" x2="6.3508" y2="6.35" width="0.8128" layer="1"/>
 </signal>
 <signal name="N$2">
