File: PLACAS/Sensors_Dev_Modules v.1.0/UVB Module.sch (EAGLE design)
At the start: 5 parts

Commit message: Add files via upload
Connections:
- net GND: now also U$1.GND; no longer U$1.GND_0, U$1.GND_1, U$1.GND_2, U$1.GND_3, U$1.GND_4
Other:
- moved on the sheet: JP2, R1, R2

Commit message: Add files via upload
Other:
- note added: "1/1"
- note added: "EESC - USP"
- note added: "Julho de 2020"
- note added: "Júlio Calandrin"
- note added: "UVB Module v.1.0"
- moved on the sheet: JP1, JP2, R1, R2
