File: PLACAS/Sensors_Dev_Modules v.1.0/UVC Module.brd (EAGLE design)
At the start: 25 x 25 mm, 12 parts, among them IC1 OPA4191ID

Commit message: Add files via upload
Connections:
- net GND: no longer U$1.GND2, U$1.GND3, U$1.GND4, U$1.GND5
Routing:
- net GND: track 82.8 -> 79.1 mm
- net UVC-CATHODE: track 18.0 -> 15.4 mm
Other:
- board text added: "UVC MODULE"
- board text removed: "UVA MODULE"

Commit message: Add files via upload
Routing:
- net 1ºESTAGIO: track 11.5 -> 20.5 mm
- net UVC: track 14.7 -> 9.69 mm
- net GND: track 79.1 -> 76.5 mm
- net -5V: track 17.1 -> 15.1 mm, vias 2 -> 1
- net +5V: track 27.5 -> 25.8 mm, vias 2 -> 1
Changed lines of the file:
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@@
 <?xml version="1.0" encoding="utf-8"?>
 <!DOCTYPE eagle SYSTEM "eagle.dtd">
-<eagle version="9.6.2">
+<eagle version="9.4.2">
 <drawing>
 <settings>
@@
 <setting verticaltext="up"/>
 </settings>
-<grid distance="0.5" unitdist="mm" unit="mm" style="dots" multiple="1" display="yes" altdistance="0.01" altunitdist="mm" altunit="mm"/>
+<grid distance="12.5" unitdist="mil" unit="mil" style="dots" multiple="1" display="yes" altdistance="0.01" altunitdist="mm" altunit="mm"/>
 <layers>
 <layer number="1" name="Top" color="4" fill="1" visible="yes" active="yes"/>
@@
 <wire x1="14.06" y1="-12.51" x2="14.9588" y2="-12.51" width="0.4064" layer="16"/>
 <contactref element="JP1" pad="1"/>
-<wire x1="15.04" y1="-21.38" x2="16.75" y2="-20.34" width="0.4064" layer="16"/>
-<wire x1="16.75" y1="-20.34" x2="16.75" y2="-18.85" width="0.4064" layer="16"/>
-<via x="16.75" y="-18.85" extent="1-16" drill="0.35"/>
-<wire x1="16.75" y1="-18.85" x2="16.75" y2="-16.75" width="0.4064" layer="1"/>
-<wire x1="16.75" y1="-16.75" x2="13.15" y2="-13.15" width="0.4064" layer="1"/>
-<wire x1="13.15" y1="-13.15" x2="13.15" y2="-12.8" width="0.4064" layer="1"/>
 <via x="13.15" y="-12.8" extent="1-16" drill="0.35"/>
 <wire x1="13.15" y1="-12.8" x2="13.44" y2="-12.51" width="0.4064" layer="16"/>
 <wire x1="13.44" y1="-12.51" x2="14.9588" y2="-12.51" width="0.4064" layer="16"/>
+<wire x1="15.04" y1="-21.38" x2="15.04" y2="-20.4375" width="0.4064" layer="1"/>
+<wire x1="13.15" y1="-18.5475" x2="13.15" y2="-12.8" width="0.4064" layer="1"/>
+<wire x1="15.04" y1="-20.4375" x2="13.15" y2="-18.5475" width="0.4064" layer="1"/>
 </signal>
 <signal name="-5V">
@@
 <wire x1="7.705" y1="-11.305" x2="8.86" y2="-12.46" width="0.508" layer="16"/>
 <contactref element="JP1" pad="3"/>
-<wire x1="9.96" y1="-21.38" x2="8" y2="-20.09" width="0.4064" layer="16"/>
-<wire x1="8" y1="-20.09" x2="8" y2="-18.8" width="0.4064" layer="16"/>
-<via x="8" y="-18.8" extent="1-16" drill="0.35"/>
-<wire x1="8" y1="-18.8" x2="8" y2="-16.95" width="0.4064" layer="1"/>
-<wire x1="11.75" y1="-13.2" x2="11.75" y2="-12.5" width="0.4064" layer="1"/>
-<via x="11.75" y="-12.5" extent="1-16" drill="0.35"/>
-<wire x1="11.75" y1="-12.5" x2="11.74" y2="-12.51" width="0.4064" layer="16"/>
-<wire x1="11.74" y1="-12.51" x2="10.0312" y2="-12.51" width="0.4064" layer="16"/>
-<wire x1="8" y1="-16.95" x2="11.75" y2="-13.2" width="0.4064" layer="1"/>
+<via x="11.75" y="-12.8175" extent="1-16" drill="0.35"/>
+<wire x1="11.75" y1="-12.8175" x2="11.4425" y2="-12.51" width="0.4064" layer="16"/>
+<wire x1="11.4425" y1="-12.51" x2="10.0312" y2="-12.51" width="0.4064" layer="16"/>
+<wire x1="9.96" y1="-21.38" x2="9.96" y2="-20.2025" width="0.4064" layer="1"/>
+<wire x1="11.75" y1="-18.4125" x2="11.75" y2="-12.8175" width="0.4064" layer="1"/>
+<wire x1="9.96" y1="-20.2025" x2="11.75" y2="-18.4125" width="0.4064" layer="1"/>
 </signal>
 <signal name="GND">
@@
 <wire x1="17.71" y1="-15.83" x2="17.61" y2="-15.73" width="0.1524" layer="16"/>
 <wire x1="20.135" y1="-15.83" x2="20.1452875" y2="-15.83" width="0.1524" layer="16"/>
-<wire x1="20.1452875" y1="-15.83" x2="21.55" y2="-14.800934375" width="0.1524" layer="16"/>
 <wire x1="10.0312" y1="-13.78" x2="8.98" y2="-13.78" width="0.1524" layer="16"/>
 <wire x1="8.98" y1="-13.78" x2="8.65" y2="-13.45" width="0.1524" layer="16"/>
@@
 <wire x1="8.65" y1="-15.05" x2="8.65" y2="-15.5" width="0.1524" layer="16"/>
 <wire x1="8.65" y1="-15.5" x2="8.85" y2="-15.7" width="0.1524" layer="16"/>
-<wire x1="11.55" y1="-15.4" x2="11.55" y2="-13.9" width="0.1524" layer="16"/>
-<wire x1="11.55" y1="-13.9" x2="11.43" y2="-13.78" width="0.1524" layer="16"/>
-<wire x1="11.43" y1="-13.78" x2="10.0312" y2="-13.78" width="0.1524" layer="16"/>
+<wire x1="11.55" y1="-15.4" x2="11.55" y2="-14.535" width="0.1524" layer="16"/>
+<wire x1="11.55" y1="-14.535" x2="10.795" y2="-13.78" width="0.1524" layer="16"/>
+<wire x1="10.795" y1="-13.78" x2="10.0312" y2="-13.78" width="0.1524" layer="16"/>
 <wire x1="8.85" y1="-15.7" x2="11.25" y2="-15.7" width="0.1524" layer="16"/>
 <wire x1="11.25" y1="-15.7" x2="11.55" y2="-15.4" width="0.1524" layer="16"/>
@@
 <wire x1="16.5" y1="-14.85" x2="16.5" y2="-15.5" width="0.1524" layer="16"/>
 <wire x1="16.5" y1="-15.5" x2="16.83" y2="-15.83" width="0.1524" layer="16"/>
-<wire x1="22.55" y1="-11.2" x2="21.45" y2="-10.1" width="0.1524" layer="16"/>
-<wire x1="21.45" y1="-10.1" x2="16.9" y2="-10.1" width="0.1524" layer="16"/>
+<wire x1="22.55" y1="-10.7" x2="21.95" y2="-10.1" width="0.1524" layer="16"/>
+<wire x1="21.95" y1="-10.1" x2="16.9" y2="-10.1" width="0.1524" layer="16"/>
 <wire x1="16.9" y1="-10.1" x2="16.15" y2="-9.35" width="0.1524" layer="16"/>
-<wire x1="22.55" y1="-11.2" x2="22.55" y2="-11.9" width="0.1524" layer="16"/>
+<wire x1="22.55" y1="-10.7" x2="22.55" y2="-11.9" width="0.1524" layer="16"/>
 <wire x1="16.15" y1="-9.35" x2="13.9" y2="-9.35" width="0.1524" layer="16"/>
 <wire x1="13.9" y1="-9.35" x2="13.35" y2="-9.9" width="0.1524" layer="16"/>
@@
 <wire x1="21.95" y1="-12.5" x2="21.45" y2="-12.5" width="0.1524" layer="16"/>
 <wire x1="21.45" y1="-12.5" x2="16.8" y2="-12.5" width="0.1524" layer="16"/>
-<wire x1="21.55" y1="-14.800934375" x2="21.95" y2="-14.400934375" width="0.1524" layer="16"/>
-<wire x1="21.95" y1="-14.400934375" x2="21.95" y2="-13" width="0.1524" layer="16"/>
-<wire x1="21.95" y1="-13" x2="21.95" y2="-12.5" width="0.1524" layer="16"/>
-<wire x1="21.95" y1="-13" x2="21.45" y2="-12.5" width="0.1524" layer="16"/>
 <polygon width="0.1524" layer="1">
 <vertex x="-0.5" y="0.5"/>
@@
 <contactref element="U$1" pad="GND1"/>
 <contactref element="U$1" pad="GND0"/>
+<wire x1="17.71" y1="-15.83" x2="20.135" y2="-15.83" width="0.1524" layer="16"/>
 </signal>
 <signal name="UVC-CATHODE">
@@
 <wire x1="17.61" y1="-11.15" x2="17.71" y2="-11.05" width="0.508" layer="16"/>
 <wire x1="17.71" y1="-11.05" x2="20.135" y2="-11.05" width="0.508" layer="16"/>
-<wire x1="20.135" y1="-11.05" x2="21.4" y2="-11.05" width="0.4064" layer="16"/>
-<wire x1="21.4" y1="-11.05" x2="21.8" y2="-11.45" width="0.4064" layer="16"/>
-<via x="21.8" y="-11.45" extent="1-16" drill="0.35"/>
+<wire x1="20.135" y1="-11.05" x2="21.65" y2="-11.05" width="0.4064" layer="16"/>
+<wire x1="21.65" y1="-11.05" x2="21.8" y2="-11.2" width="0.4064" layer="16"/>
+<via x="21.8" y="-11.2" extent="1-16" drill="0.35"/>
 <contactref element="U$1" pad="SINAL2"/>
 <contactref element="U$1" pad="SINAL1"/>
 <wire x1="17.5" y1="-13.77" x2="17.5" y2="-11.23" width="0.8128" layer="1"/>
-<wire x1="17.5" y1="-11.23" x2="21.58" y2="-11.23" width="0.6096" layer="1"/>
-<wire x1="21.58" y1="-11.23" x2="21.8" y2="-11.45" width="0.6096" layer="1"/>
+<wire x1="17.5" y1="-11.23" x2="21.77" y2="-11.23" width="0.6096" layer="1"/>
+<wire x1="21.77" y1="-11.23" x2="21.8" y2="-11.2" width="0.6096" layer="1"/>
 </signal>
 <signal name="3ºESTAGIO">
@@
 <wire x1="17.56" y1="-13.78" x2="17.71" y2="-13.93" width="0.508" layer="16"/>
 <wire x1="17.71" y1="-13.93" x2="20.135" y2="-13.93" width="0.508" layer="16"/>
-<wire x1="17.788" y1="-13.458" x2="17.71" y2="-9.15" width="0" layer="19" extent="16-16"/>
+<wire x1="20.135" y1="-9.15" x2="21.85" y2="-9.15" width="0.508" layer="16"/>
+<wire x1="21.85" y1="-9.15" x2="23.1775" y2="-10.4775" width="0.508" layer="16"/>
+<wire x1="21.3125" y1="-13.93" x2="20.135" y2="-13.93" width="0.508" layer="16"/>
+<wire x1="23.1775" y1="-10.4775" x2="23.1775" y2="-12.065" width="0.508" layer="16"/>
+<wire x1="23.1775" y1="-12.065" x2="21.3125" y2="-13.93" width="0.508" layer="16"/>
 </signal>
 <signal name="2ºESTAGIO">
@@
 <wire x1="11.78" y1="-9.97" x2="11.8" y2="-9.95" width="0.4064" layer="16"/>
 <via x="11.8" y="-9.95" extent="1-16" drill="0.35"/>
-<wire x1="11.8" y1="-9.95" x2="10.05" y2="-9.95" width="0.4064" layer="1"/>
-<wire x1="10.05" y1="-9.95" x2="8.5" y2="-8.4" width="0.4064" layer="1"/>
-<wire x1="8.5" y1="-8.4" x2="8.5" y2="-6.38" width="0.4064" layer="1"/>
-<wire x1="9.28" y1="-5.6" x2="11.4" y2="-5.6" width="0.4064" layer="1"/>
-<wire x1="11.4" y1="-5.6" x2="12.55" y2="-4.45" width="0.4064" layer="1"/>
+<wire x1="12.5" y1="-4.5" x2="12.5" y2="-9.25" width="0.4064" layer="1"/>
+<wire x1="11.8" y1="-9.95" x2="12.5" y2="-9.25" width="0.4064" layer="1"/>
+<wire x1="12.5" y1="-4.5" x2="12.55" y2="-4.45" width="0.4064" layer="1"/>
 <wire x1="12.55" y1="-4.45" x2="12.5" y2="-3.62" width="0.4064" layer="1"/>
-<wire x1="8.5" y1="-6.38" x2="9.28" y2="-5.6" width="0.4064" layer="1"/>
 </signal>
 </signals>
