File: PLACAS/Sensors_Dev_Modules v.1.0/Módulo U.V. v.1.0.brd (EAGLE design)
At the start: 25 x 25 mm, 14 parts, among them IC3 MCP6242-E_SN

Commit message: Add files via upload
Routing:
- net GND: track 1.27 -> 0.17 mm
- net N$1: track 14.3 -> 15.0 mm
Changed lines of the file:
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@@
 <?xml version="1.0" encoding="utf-8"?>
 <!DOCTYPE eagle SYSTEM "eagle.dtd">
-<eagle version="9.4.2">
+<eagle version="9.6.2">
 <drawing>
 <settings>
@@
 <setting verticaltext="up"/>
 </settings>
-<grid distance="6.25" unitdist="mil" unit="mil" style="lines" multiple="1" display="yes" altdistance="6.25" altunitdist="mil" altunit="mil"/>
+<grid distance="0.3175" unitdist="mm" unit="mm" style="lines" multiple="1" display="yes" altdistance="6.25" altunitdist="mil" altunit="mm"/>
 <layers>
 <layer number="1" name="Top" color="4" fill="1" visible="yes" active="yes"/>
@@
 </layers>
 <board>
-<fusionsync huburn="a.cGVyc29uYWw6dWUyYWE0YjY0" projecturn="a.cGVyc29uYWw6dWUyYWE0YjY0IzIwMTkxMDIwMjI4OTQ0ODI2" f3durn="urn:adsk.wipprod:dm.lineage:8Ilb3DUWRheq4yj4YiRVXg" pcbguid="f087186c-2854-4546-a95c-53110e0ce7fa" lastpulledtime="" lastsyncedchangeguid=""/>
+<fusionsync huburn="a.cGVyc29uYWw6dWUyYWE0YjY0" projecturn="a.cGVyc29uYWw6dWUyYWE0YjY0IzIwMTkxMDIwMjI4OTQ0ODI2" f3durn="urn:adsk.wipprod:dm.lineage:8Ilb3DUWRheq4yj4YiRVXg" pcbguid="f087186c-2854-4546-a95c-53110e0ce7fa" lastpulledtime="" lastsyncedchangeguid="" latestrevisionid="" lastsyncedrevisionid="" lastboardhashguid="" lastpushedtime="" linktopcb3d="true"/>
 <plain>
 <circle x="4" y="-4" radius="3.2" width="0.4064" layer="41"/>
@@
 <contactref element="C9" pad="2"/>
 <contactref element="D1" pad="2"/>
-<wire x1="9.789" y1="-10.2775" x2="9.789" y2="-11.5475" width="0.6096" layer="16"/>
+<wire x1="10.995" y1="-11.5475" x2="11.1125" y2="-11.43" width="0.1524" layer="16"/>
 </signal>
 <signal name="UVC">
@@
 <contactref element="C10" pad="1"/>
 <wire x1="17.9825" y1="-12.8175" x2="18.0975" y2="-12.7025" width="0.508" layer="16"/>
-<wire x1="18.4175" y1="-12.7025" x2="18.0975" y2="-12.7025" width="0.508" layer="16"/>
 <wire x1="15.211" y1="-12.8175" x2="17.9825" y2="-12.8175" width="0.6096" layer="16"/>
-<wire x1="18.0975" y1="-12.7025" x2="18.57625" y2="-12.7025" width="0.6096" layer="16"/>
-<wire x1="20.47875" y1="-14.605" x2="18.57625" y2="-12.7025" width="0.6096" layer="16"/>
 <wire x1="15.04" y1="-21.38" x2="15.04" y2="-20.5175" width="0.6096" layer="16"/>
 <wire x1="15.04" y1="-20.5175" x2="20.955" y2="-14.6025" width="0.6096" layer="16"/>
 <wire x1="20.955" y1="-14.6025" x2="20.9525" y2="-14.605" width="0.6096" layer="16"/>
 <wire x1="20.9525" y1="-14.605" x2="20.47875" y2="-14.605" width="0.6096" layer="16"/>
+<wire x1="18.0975" y1="-12.7025" x2="18.4175" y2="-12.7025" width="0.6096" layer="16"/>
+<wire x1="20.3175" y1="-14.6025" x2="20.955" y2="-14.6025" width="0.6096" layer="16"/>
+<wire x1="18.4175" y1="-12.7025" x2="20.3175" y2="-14.6025" width="0.6096" layer="16"/>
 </signal>
 <signal name="N$6">
@@
 <wire x1="3.65375" y1="-10.475" x2="3.96875" y2="-10.475" width="0.508" layer="16"/>
 <wire x1="3.4925" y1="-10.63625" x2="3.65375" y2="-10.475" width="0.508" layer="16"/>
-<wire x1="6.82625" y1="-14.6025" x2="7.34125" y2="-14.0875" width="0.6096" layer="16"/>
-<wire x1="7.34125" y1="-14.0875" x2="9.789" y2="-14.0875" width="0.6096" layer="16"/>
+<wire x1="6.82625" y1="-14.6025" x2="7.02375" y2="-14.405" width="0.6096" layer="16"/>
+<wire x1="9.4715" y1="-14.405" x2="9.789" y2="-14.0875" width="0.6096" layer="16"/>
+<wire x1="9.4715" y1="-14.405" x2="7.02375" y2="-14.405" width="0.6096" layer="16"/>
 <wire x1="3.96875" y1="-14.6025" x2="6.6675" y2="-14.6025" width="0.6096" layer="16"/>
-<wire x1="3.96875" y1="-14.6025" x2="3.64875" y2="-14.6025" width="0.6096" layer="16"/>
-<wire x1="3.64875" y1="-14.6025" x2="2.54" y2="-13.49375" width="0.6096" layer="16"/>
-<wire x1="2.54" y1="-11.58875" x2="3.4925" y2="-10.63625" width="0.6096" layer="16"/>
-<wire x1="2.54" y1="-13.49375" x2="2.54" y2="-11.58875" width="0.6096" layer="16"/>
+<wire x1="3.96875" y1="-14.6025" x2="3.1725" y2="-14.6025" width="0.6096" layer="16"/>
+<wire x1="3.1725" y1="-14.6025" x2="2.2225" y2="-13.6525" width="0.6096" layer="16"/>
+<wire x1="3.175" y1="-10.63625" x2="3.4925" y2="-10.63625" width="0.6096" layer="16"/>
+<wire x1="3.175" y1="-10.63625" x2="2.2225" y2="-11.58875" width="0.6096" layer="16"/>
+<wire x1="2.2225" y1="-13.6525" x2="2.2225" y2="-11.58875" width="0.6096" layer="16"/>
 </signal>
 <signal name="SDA/SINAL">
@@
 <wire x1="11.23" y1="-18.77375" x2="11.23" y2="-17.5" width="0.6096" layer="1"/>
 <wire x1="9.96" y1="-20.04375" x2="11.23" y2="-18.77375" width="0.6096" layer="1"/>
-<wire x1="11.23" y1="-17.5" x2="6.82625" y2="-13.09625" width="0.6096" layer="1"/>
+<wire x1="11.23" y1="-17.5" x2="7.18375" y2="-13.45375" width="0.6096" layer="1"/>
+<wire x1="7.18375" y1="-13.45375" x2="6.82625" y2="-13.09625" width="0.6096" layer="1"/>
 <wire x1="6.82625" y1="-13.09625" x2="6.82625" y2="-11.43" width="0.6096" layer="1"/>
 <wire x1="6.82625" y1="-11.43" x2="6.82625" y2="-12.7025" width="0.6096" layer="16"/>
