File: PLACAS/Sensors_Dev_Modules v.1.0/Módulo U.V.C. v.1.0.brd (EAGLE design)
At the start: 25 x 25 mm, 12 parts, among them IC1 OPA4191ID

Commit message: Add files via upload
Parts:
- removed U$1: (no value), Zenith_Breakouts:PADS_UV-C
- added U$3: UNIVERSAL_BREAKOUT, Zenith_Breakouts:UNIVERSAL_PADS
Connections:
- net GND: now also U$3.GND; no longer U$1.GND0, U$1.GND1
- net UVC-CATHODE: now also U$3.SDA/SINAL; no longer U$1.SINAL1, U$1.SINAL2
Routing:
- net UVC-CATHODE: track 20.3 -> 17.7 mm
- net GND: track 59.3 -> 61.1 mm
