File: PLACAS/Sensors_Dev_Modules v.1.0/Módulo U.V.C. v.1.0.sch (EAGLE design)
At the start: 12 parts, among them IC1 OPA4191ID

Commit message: Add files via upload
Parts:
- removed U$1: (no value), Zenith_Breakouts:BREAKOUT_UV-C
- added U$3: UNIVERSAL_BREAKOUT, Zenith_Breakouts:UNIVERSAL_BREAKOUT
Connections:
- net GND: now also U$3.GND; no longer U$1.GND_0, U$1.GND_1
- net UVC-CATHODE: now also U$3.SDA/SINAL; no longer U$1.SINAL_1, U$1.SINAL_2
Changed lines of the file:
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@@
 <?xml version="1.0" encoding="utf-8"?>
 <!DOCTYPE eagle SYSTEM "eagle.dtd">
-<eagle version="9.4.2">
+<eagle version="9.6.2">
 <drawing>
 <settings>
@@
 <part name="P+2" library="supply1" library_urn="urn:adsk.eagle:library:371" deviceset="+5V" device=""/>
 <part name="P-2" library="supply1" library_urn="urn:adsk.eagle:library:371" deviceset="-5V" device=""/>
-<part name="U$1" library="Zenith_Breakouts" deviceset="BREAKOUT_UV-C" device=""/>
 <part name="FRAME1" library="frames" library_urn="urn:adsk.eagle:library:229" deviceset="A4L-LOC" device=""/>
+<part name="U$3" library="Zenith_Breakouts" deviceset="UNIVERSAL_BREAKOUT" device=""/>
 </parts>
 <sheets>
@@
 <attribute name="VALUE" x="68.58" y="78.74" size="1.778" layer="96" rot="R180"/>
 </instance>
-<instance part="U$1" gate="G$1" x="68.58" y="139.7" smashed="yes" rot="R90"/>
 <instance part="FRAME1" gate="G$1" x="-0.7" y="-0.3" smashed="yes"/>
+<instance part="U$3" gate="G$1" x="78.74" y="139.7" smashed="yes" rot="R90"/>
 </instances>
 <busses>
@@
 <wire x1="116.84" y1="121.92" x2="124.46" y2="121.92" width="0.1524" layer="91"/>
 <wire x1="116.84" y1="114.3" x2="116.84" y2="116.84" width="0.1524" layer="91"/>
+<pinref part="U$3" gate="G$1" pin="GND"/>
 <wire x1="116.84" y1="116.84" x2="116.84" y2="121.92" width="0.1524" layer="91"/>
+<wire x1="81.28" y1="127" x2="81.28" y2="116.84" width="0.1524" layer="91"/>
+<wire x1="81.28" y1="116.84" x2="116.84" y2="116.84" width="0.1524" layer="91"/>
 <junction x="116.84" y="116.84"/>
-<pinref part="U$1" gate="G$1" pin="GND_1"/>
-<wire x1="68.58" y1="116.84" x2="116.84" y2="116.84" width="0.1524" layer="91"/>
-<wire x1="66.04" y1="127" x2="66.04" y2="124.46" width="0.1524" layer="91"/>
-<wire x1="66.04" y1="124.46" x2="68.58" y2="124.46" width="0.1524" layer="91"/>
-<pinref part="U$1" gate="G$1" pin="GND_0"/>
-<wire x1="68.58" y1="124.46" x2="71.12" y2="124.46" width="0.1524" layer="91"/>
-<wire x1="71.12" y1="124.46" x2="71.12" y2="127" width="0.1524" layer="91"/>
-<wire x1="68.58" y1="124.46" x2="68.58" y2="116.84" width="0.1524" layer="91"/>
-<junction x="68.58" y="124.46"/>
 </segment>
 <segment>
@@
 <junction x="116.84" y="127"/>
 <pinref part="R4" gate="G$1" pin="1"/>
-<wire x1="68.58" y1="154.94" x2="68.58" y2="162.56" width="0.1524" layer="91"/>
-<wire x1="68.58" y1="162.56" x2="111.76" y2="162.56" width="0.1524" layer="91"/>
+<wire x1="81.28" y1="162.56" x2="111.76" y2="162.56" width="0.1524" layer="91"/>
 <wire x1="111.76" y1="162.56" x2="111.76" y2="127" width="0.1524" layer="91"/>
 <junction x="111.76" y="127"/>
-<pinref part="U$1" gate="G$1" pin="SINAL_2"/>
-<wire x1="66.04" y1="152.4" x2="66.04" y2="154.94" width="0.1524" layer="91"/>
-<wire x1="66.04" y1="154.94" x2="68.58" y2="154.94" width="0.1524" layer="91"/>
-<pinref part="U$1" gate="G$1" pin="SINAL_1"/>
-<wire x1="68.58" y1="154.94" x2="71.12" y2="154.94" width="0.1524" layer="91"/>
-<wire x1="71.12" y1="154.94" x2="71.12" y2="152.4" width="0.1524" layer="91"/>
-<junction x="68.58" y="154.94"/>
+<pinref part="U$3" gate="G$1" pin="SDA/SINAL"/>
+<wire x1="81.28" y1="152.4" x2="81.28" y2="162.56" width="0.1524" layer="91"/>
 </segment>
 </net>
