File: PLACAS/Varella_Std v.2.0/Varella_Std - v.2.0.sch (EAGLE design)
At the start: 92 parts, among them IC1 74HC4051D,653, IC3 M95M04-DRDW6TP, IC4 M95M04-DRDW6TP, IC5 M95M04-DRDW6TP, IC6 M95M04-DRDW6TP, IC7 TESEO-LIV3F, IC8 BGA_725L6_E6327, U1 MAX31856, U2 MAX31856, U3 MAX31856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

Commit message: Add files via upload
Parts:
- removed C26, C27: (no value), rcl:C-EUC0805
- removed SJ2, SJ3, SJ4, SJ5: (no value), FaBo-PIN:SMD-JUMPER-2
- removed U$7: CRYSTAL, cristal:CRYSTAL
- added C42: 56pF, rcl:C-EUC1206
- added C43: 22uF, rcl:C-EUC1206
- added C54, C55: 10pF, rcl:C-EUC0805
- added IC13: ST1S12GR, SamacSys_Parts:ST1S12GR
- added MCO, RX_CODE, TX_CODE: (no value), FaBo-PIN:SMD-JUMPER-2
- added R29: 1M, rcl (2):R-EU_M1206
- added R30: 68k, rcl (2):R-EU_M1206
- added R31: 27k, rcl (2):R-EU_M1206
- added U$2: LTF5022T100M1R4, LTF5022T:LTF5022T100M1R4
- added Y5: FA-20H_16.0000MF10Z-AJ0, SamacSys_Parts:FA-20H_16.0000MF10Z-AJ0
- C16, C17, C18, C19, C20: value (none) -> 100nF
- C21: value (none) -> 1uF
- C22: value (none) -> 0,1uF
- C23, C24: value (none) -> 10pF
- R10: value (none) -> 220
- R11, R12, R15, R16, R17, R18, R19, R20, R21, R22: value (none) -> 4,7k
- R8, R9: value (none) -> 1k
Connections:
- net SDA1/UART_TX renamed SDA1/UART_RX
- net SDA2/UART_RX renamed SDA2/UART_TX
- removed net SCL_NEOM8: SJ3.1, U$3.19_SCL/SPI_CLK
- removed net SCL_TESEO: IC7.SCL, SJ5.1
- removed net SDA_NEOM8: SJ2.1, U$3.18_SDA/SPI_CS_N
- removed net SDA_TESEO: IC7.SDA, SJ4.1
- new net N$37: IC13.EN, R29.1
- new net N$38: IC13.SW, U$2.1
- new net N$39: IC13.FB/VO, R30.1, R31.2
- new net TESEO3: C30.1, C43.1, L4-27NH.1, R30.2, U$2.2
- new net UART_RX_CODE: CODE_UPLOAD-3.S, RX_CODE.2
- new net UART_TX_CODE: CODE_UPLOAD-4.S, TX_CODE.2
- net +3V3: now also C42.1, IC13.VIN, R29.2; no longer C30.1, L4-27NH.1
- net GND: now also C42.2, C43.2, C54.2, C55.2, IC13.GND, R31.1, Y5.GND_1, Y5.GND_2; no longer C26.2, C27.2, U$7.P$1
- net MCO: now also MCO.2
- net OSC_IN: now also C54.1, MCO.1, Y5.CRYSTAL_2; no longer C26.1, U$7.1
- net OSC_OUT: now also C55.1, Y5.CRYSTAL_1; no longer C27.1, U$7.2
- net SCL4: now also IC7.SCL, U$3.19_SCL/SPI_CLK; no longer SJ3.2, SJ5.2
- net SDA4: now also IC7.SDA, U$3.18_SDA/SPI_CS_N; no longer SJ2.2, SJ4.2
- net UART_RX: now also RX_CODE.1, UART_TX.2; no longer UART_RX.2
- net UART_TX: now also TX_CODE.1, UART_RX.2; no longer UART_TX.2
Other:
- moved on the sheet: 3V3, C28, C29, C30, C31, IC7, IC8, L2-7,5NH, L4-27NH, R2, R23, X4

Commit message: Add files via upload
Parts:
- removed C16: 100nF, rcl:C-EUC0805
- removed CAN3: SN65HVD233D, SN65HVD233D:SN65HVD233D
- removed COMM_MICRO1: STM32L496RGT6, STM32L4xxx:STM32L496RGT6
- removed L2-7,5NH: 0603CS-7N5XGLU, SamacSys_Parts:0603CS-7N5XGLU
- removed MCO: (no value), FaBo-PIN:SMD-JUMPER-2
- removed VARELLA_MODULE: 53398-09, con-molex:53398-09
- added CAN: SN65HVD233D, SN65HVD233D:SN65HVD233D
- added COMM_MICRO: STM32L496RGT6, STM32L4xxx:STM32L496RGT6
- added L1: LQW18AS7N5J0ZD-7,5nH, LQW18AS7N5J0ZD:LQW18AS7N5J0ZD
- added VARELLA_AQUISITIO_MODULE: 53261-12, con-molex:53261-12
- CODE_UPLOAD: value 53398-10 -> 53261-10; device con-molex:53398-10 -> con-molex:53261-10
Connections:
- net N$2 renamed L3
- removed net MCO: CODE_UPLOAD-9.S, MCO.2
- net !DRDY_1: now also COMM_MICRO.PA9; no longer COMM_MICRO1.PA9
- net !DRDY_2: now also COMM_MICRO.PB0; no longer COMM_MICRO1.PB0
- net !DRDY_3: now also COMM_MICRO.PB1; no longer COMM_MICRO1.PB1
- net !FAULT_1: now also COMM_MICRO.PA8; no longer COMM_MICRO1.PA8
- net !FAULT_2: now also COMM_MICRO.PB2; no longer COMM_MICRO1.PB2
- net !FAULT_3: now also COMM_MICRO.PC5; no longer COMM_MICRO1.PC5
- net !HOLD: now also COMM_MICRO.PB15; no longer COMM_MICRO1.PB15
- net !W: now also COMM_MICRO.PB14; no longer COMM_MICRO1.PB14
- net +3V3: now also CAN.VCC, COMM_MICRO.VBAT, COMM_MICRO.VDD@1, COMM_MICRO.VDD@2, COMM_MICRO.VDD@4, COMM_MICRO.VDDA/VREF_PLUS, COMM_MICRO.VDDUSB, VARELLA_AQUISITIO_MODULE-7.S; no longer C16.1, CAN3.VCC, COMM_MICRO1.VBAT, COMM_MICRO1.VDD@1, COMM_MICRO1.VDD@2, COMM_MICRO1.VDD@4, COMM_MICRO1.VDDA/VREF_PLUS, COMM_MICRO1.VDDUSB, VARELLA_MODULE-3.S
- net +5V: now also VARELLA_AQUISITIO_MODULE-8.S; no longer VARELLA_MODULE-1.S
- net BOOT: now also COMM_MICRO.PH3/BOOT0; no longer COMM_MICRO1.PH3/BOOT0
- net CAN1_LBK: now also CAN.LBK, COMM_MICRO.PC7; no longer CAN3.LBK, COMM_MICRO1.PC7
- net CAN1_RX: now also CAN.RXD, COMM_MICRO.PA11; no longer CAN3.RXD, COMM_MICRO1.PA11
- net CAN1_TX: now also CAN.TXD, COMM_MICRO.PA12; no longer CAN3.TXD, COMM_MICRO1.PA12
- net CAN_H: now also CAN.CANH, VARELLA_AQUISITIO_MODULE-12.S; no longer CAN3.CANH, VARELLA_MODULE-4.S
- net CAN_L: now also CAN.CANL, VARELLA_AQUISITIO_MODULE-11.S; no longer CAN3.CANL, VARELLA_MODULE-5.S
- net EXT_INTERRUPT_NEOM8: now also COMM_MICRO.PC13; no longer COMM_MICRO1.PC13
- net EXT_INTERRUPT_TESEO: now also COMM_MICRO.PB6; no longer COMM_MICRO1.PB6
- net GND: now also CAN.GND, COMM_MICRO.VSS@1, COMM_MICRO.VSS@2, COMM_MICRO.VSS@3, COMM_MICRO.VSS@4, COMM_MICRO.VSSA/VREF_MINUS, VARELLA_AQUISITIO_MODULE-10.S, VARELLA_AQUISITIO_MODULE-9.S; no longer C16.2, CAN3.GND, COMM_MICRO1.VSS@1, COMM_MICRO1.VSS@2, COMM_MICRO1.VSS@3, COMM_MICRO1.VSS@4, COMM_MICRO1.VSSA/VREF_MINUS, VARELLA_MODULE-2.S
- net MISO_BUS: now also COMM_MICRO.PA6; no longer COMM_MICRO1.PA6
- net MISO_SENSOR: now also COMM_MICRO.PC2, VARELLA_AQUISITIO_MODULE-1.S; no longer COMM_MICRO1.PC2, VARELLA_MODULE-7.S
- net MOSI_BUS: now also COMM_MICRO.PB5; no longer COMM_MICRO1.PB5
- net MOSI_SENSOR: now also COMM_MICRO.PC3, VARELLA_AQUISITIO_MODULE-3.S; no longer COMM_MICRO1.PC3, VARELLA_MODULE-8.S
- net N$11: now also COMM_MICRO.PC6; no longer COMM_MICRO1.PC6
- net N$13: now also COMM_MICRO.PC14-OSC32-IN; no longer COMM_MICRO1.PC14-OSC32-IN
- net N$14: now also COMM_MICRO.PC15-OSC32-OUT; no longer COMM_MICRO1.PC15-OSC32-OUT
- net N$17: now also CAN.RS; no longer CAN3.RS
- net N$18: now also L1.2; no longer L2-7,5NH.2
- net N$19: now also L1.1; no longer L2-7,5NH.1
- net NRST: now also COMM_MICRO.NRST; no longer COMM_MICRO1.NRST
- net NSS_BUS: now also COMM_MICRO.PA4; no longer COMM_MICRO1.PA4
- net OSC_IN: now also CODE_UPLOAD-9.S, COMM_MICRO.PH0-OSC-IN; no longer COMM_MICRO1.PH0-OSC-IN, MCO.1
- net OSC_OUT: now also COMM_MICRO.PH1-OSC-OUT; no longer COMM_MICRO1.PH1-OSC-OUT
- net PPS_NEOM8: now also COMM_MICRO.PA0; no longer COMM_MICRO1.PA0
- net PPS_TESEO: now also COMM_MICRO.PA15; no longer COMM_MICRO1.PA15
- net RESET_NEOM8: now also COMM_MICRO.PA10; no longer COMM_MICRO1.PA10
- net RESET_TESEO: now also COMM_MICRO.PB9; no longer COMM_MICRO1.PB9
- net S0: now also COMM_MICRO.PB12; no longer COMM_MICRO1.PB12
- net S1: now also COMM_MICRO.PC4; no longer COMM_MICRO1.PC4
- net S2: now also COMM_MICRO.PA5; no longer COMM_MICRO1.PA5
- net SCL1: now also COMM_MICRO.PB8; no longer COMM_MICRO1.PB8
- net SCL2: now also COMM_MICRO.PA7; no longer COMM_MICRO1.PA7
- net SCL3: now also COMM_MICRO.PC0; no longer COMM_MICRO1.PC0
- net SCL4: now also COMM_MICRO.PB10, VARELLA_AQUISITIO_MODULE-5.S; no longer COMM_MICRO1.PB10
- net SCLK_BUS: now also COMM_MICRO.PA1; no longer COMM_MICRO1.PA1
- net SCLK_SENSOR: now also COMM_MICRO.PB13, VARELLA_AQUISITIO_MODULE-2.S; no longer COMM_MICRO1.PB13, VARELLA_MODULE-6.S
- net SDA1: now also COMM_MICRO.PB7; no longer COMM_MICRO1.PB7
- net SDA2: now also COMM_MICRO.PB4; no longer COMM_MICRO1.PB4
- net SDA3: now also COMM_MICRO.PC1; no longer COMM_MICRO1.PC1
- net SDA4: now also COMM_MICRO.PB11, VARELLA_AQUISITIO_MODULE-6.S; no longer COMM_MICRO1.PB11
- net SDMMC_CK: now also COMM_MICRO.PC12; no longer COMM_MICRO1.PC12
- net SDMMC_CMD: now also COMM_MICRO.PD2; no longer COMM_MICRO1.PD2
- net SDMMC_D0: now also COMM_MICRO.PC8; no longer COMM_MICRO1.PC8
- net SDMMC_D1: now also COMM_MICRO.PC9; no longer COMM_MICRO1.PC9
- net SDMMC_D2: now also COMM_MICRO.PC10; no longer COMM_MICRO1.PC10
- net SDMMC_D3: now also COMM_MICRO.PC11; no longer COMM_MICRO1.PC11
- net SWCLK: now also COMM_MICRO.PA14; no longer COMM_MICRO1.PA14
- net SWDIO: now also COMM_MICRO.PA13; no longer COMM_MICRO1.PA13
- net SWO: now also COMM_MICRO.PB3; no longer COMM_MICRO1.PB3
- net UART_RX: now also COMM_MICRO.PA3; no longer COMM_MICRO1.PA3
- net UART_TX: now also COMM_MICRO.PA2; no longer COMM_MICRO1.PA2
- net Y3: now also VARELLA_AQUISITIO_MODULE-4.S; no longer VARELLA_MODULE-9.S
Other:
- note added: "EEPROM"
- note added: "NEO-M8Q"
- note added: "TESEO-LIV3F"
- moved on the sheet: 3V3, C1, C10, C11, C12, C13, C14, C15, C17, C18, C19, C2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

Commit message: Add files via upload
Parts:
- added R24, R25: 4,7k, rcl:R-EU_R0805
Connections:
- net +3V3: now also R24.2, R25.2
- net SCL4: now also R24.1
- net SDA4: now also R25.1
Other:
- note added: "1/2"
- note added: "2/2"
- note added: "EESC - USP"
- note added: "João Marcus E. Morais de Assunção e Giovana Martins Losacco"
- note added: "Julho de 2020"
- note added: "Microcontrolador"
- note added: "Pull - Up I2C"
- note removed: "Microcontroller"
- moved on the sheet: I2C1, I2C2, IC1, MICROSD_CARD, R11, R18, R19, R20, R21, R22, R8, SJ1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
