File: PLACAS/Varella_Std v.2.0/Varella_Std - v.2.0.sch (EAGLE design)
At the start: 98 parts, among them IC1 74HC4051D,653, IC13 ST1S12GR, IC3 M95M04-DRDW6TP, IC4 M95M04-DRDW6TP, IC5 M95M04-DRDW6TP, IC6 M95M04-DRDW6TP, IC7 TESEO-LIV3F, IC8 BGA_725L6_E6327, U1 MAX31856, U2 MAX31856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

Commit message: Add files via upload
Parts:
- C30: value 1onF -> 10nF
- renumbered VARELLA_AQUISITIO_MODULE to VARELLA_AQUISITION_MODULE
