File: PLACAS/Varella_Aquisition_Module v.2.0/Varella_Aquisition_Module - v.2.0.brd (EAGLE design)
At the start: 100 x 80 mm, 62 parts, among them IC1 M95M04-DRDW6TP, IC10 ICL7660SCBAZ, IC3 M95M04-DRDW6TP, IC4 M95M04-DRDW6TP, IC9 M95M04-DRDW6TP, U1 FT232RLSSOP, X2 USB-SMD-NS, Y2 FA-20H_16.0000MF10Z-AJ0

Commit message: Add files via upload
Parts:
- added R24, R25: 4,7k, rcl:R0805
Connections:
- net +3V3: now also R24.2, R25.2
- net SCL3: now also R24.1
- net SDA3: now also R25.1
Routing:
- net SCL3: track 61.7 -> 69.6 mm, vias 1 -> 2
- net SDA3: track 64.2 -> 71.3 mm, vias 1 -> 2

Commit message: Add files via upload
Parts:
- removed U$1: UVA_MODULE, Zenith_Breakouts:UVA_MODULE
- removed U$4: UVB_MODULE, Zenith_Breakouts:UVB_MODULE
- removed U$5: UVC_MODULE, Zenith_Breakouts:UVC_MODULE
- added 3V3, 5V: (no value), FaBo-PIN:SMD-JUMPER-2
- added R1, R2, R5, R6: 4,7k, rcl:R0805
- added U$6, U$7, U$8: MODULO_UV, Zenith_Breakouts:MODULO_UV
- C1, C11: value 0.1uF -> 100nF
- C20: value 0,1uF -> 100nF
- R19, R20, R22: value 1K -> 1k
- RX2: value Green -> (none)
- TX2: value Red -> (none)
- moved C37 14.1 mm to (81.0, 23.7)
- moved C38 14.0 mm to (95.1, 23.7), turned to 0 degrees
- turned IC10 to 90 degrees
Connections:
- removed net -5V: C38.1, IC10.5, U$5.4
- new net V+: 3V3.1, 5V.1, IC10.8, U$8.4
- new net V-: C38.1, IC10.5, U$8.6
- net +3V3: now also 3V3.2, R1.2, R2.2, R5.2, R6.2, U$6.4, U$7.4; no longer U$1.2, U$4.2
- net +5V: now also 5V.2; no longer IC10.8, U$5.6
- net GND: now also U$6.5, U$7.5, U$8.5; no longer U$1.1, U$1.3, U$1.5, U$4.1, U$4.3, U$4.5, U$5.1, U$5.3, U$5.5
- net SCL1: now also R5.1, U$6.2; no longer U$1.6
- net SCL2: now also R1.1, U$7.2; no longer U$4.6
- net SDA1: now also R6.1, U$6.1; no longer U$1.4
- net SDA2: now also R2.1, U$7.1; no longer U$4.4
- net UVC: now also U$8.3; no longer U$5.2
Routing:
- net +3V3: track 422.1 -> 487.9 mm, vias 14 -> 17
- net V+: track 0.00 -> 28.1 mm
- net +5V: track 159.1 -> 140.7 mm
- net SDA2: track 25.0 -> 42.8 mm
- net SCL2: track 30.4 -> 46.9 mm
- net SDA1: track 115.8 -> 131.7 mm
- net SCL1: track 117.3 -> 132.3 mm
- net -5V: track 11.1 -> 0.00 mm
- net V-: track 0.00 -> 10.2 mm
- net N$13: track 14.3 -> 8.36 mm
- net UVC: track 33.8 -> 39.6 mm
- net N$12: track 5.76 -> 10.8 mm
- net SCL3: track 69.6 -> 67.7 mm
- net SDA3: track 71.3 -> 70.4 mm
- net MOSI_BUS: track 48.5 -> 47.9 mm
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
Commit message: Add files via upload
Parts:
- removed CAN1: SN65HVD233D, SN65HVD233D:SOIC8
- removed LED5, LED6, LED7, LED8: TLLG4400-AS12, SamacSys_Parts:TLLG4400AS12
- removed RX2, TX2: (no value), led:CHIPLED_0805
- added CAN: SN65HVD233D, SN65HVD233D:SOIC8
- added LED1, LED2, LED3, LED4: TLLG4400-AS12, SamacSys_Parts:TLLG4400AS12
- added RX, TX: (no value), led:CHIPLED_0805
- moved C20 14.1 mm to (56.6, 10.9)
- moved COMM_MICRO2 14.1 mm to (46.7, 25.4)
- moved IC3 14.1 mm to (57.4, 41.4)
- moved R29 14.1 mm to (57.4, 35.6)
- moved R6 14.1 mm to (61.9, 58.1)
- moved U$2 14.1 mm to (2.01, 64.0)
- moved U$3 14.1 mm to (34.0, 55.6)
- moved 3V3 14.1 mm to (92.2, 9.84)
- moved 5V 14.1 mm to (92.2, 12.4)
- moved C11 14.1 mm to (25.9, 13.9)
- moved C18 14.1 mm to (37.1, 19.2)
- moved C2 14.1 mm to (25.3, 20.7)
- moved C3 14.1 mm to (3.00, 42.2)
- moved C32 14.1 mm to (32.6, 19.2)
- moved C33 14.1 mm to (32.6, 10.7)
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Connections:
- net +3V3: now also CAN.3, LED4.1; no longer CAN1.3, LED8.1
- net CAN1_LBK: now also CAN.5; no longer CAN1.5
- net CAN1_RX: now also CAN.4; no longer CAN1.4
- net CAN1_TX: now also CAN.1; no longer CAN1.1
- net CAN_H: now also CAN.7; no longer CAN1.7
- net CAN_L: now also CAN.6; no longer CAN1.6
- net GND: now also CAN.2; no longer CAN1.2
- net LED_DEBUG: now also LED3.1; no longer LED7.1
- net LED_SD: now also LED1.1; no longer LED5.1
- net LED_USB: now also LED2.1; no longer LED6.1
- net N$11: now also CAN.8; no longer CAN1.8
- net N$16: now also LED1.2; no longer LED5.2
- net N$17: now also LED2.2; no longer LED6.2
- net N$19: now also LED3.2; no longer LED7.2
- net N$20: now also LED4.2; no longer LED8.2
- net RXL: now also RX.A; no longer RX2.A
- net RXLED: now also RX.C; no longer RX2.C
- net TXL: now also TX.A; no longer TX2.A
- net TXLED: now also TX.C; no longer TX2.C
Routing:
- net +3V3: track 487.9 -> 487.3 mm
- net MISO_MEMORY: track 62.1 -> 62.6 mm
Other:
- board text added: "C:/Users/marcu/Desktop/zenith-v3.bmp"
- board text added: "Varella Aquisition Module"
- board text removed: "Varella_Aquisition_Module"
